File: Single_transistor_AMP/Single_transistor_AMP_miculis.sch (KiCad schematic (older format))
At the start: 10 parts, among them J1 Conn_01x02, J2 Conn_01x02, Q1 BC548

Commit message: Majas darbi
Parts:
- C1, C3: value 20uF -> 22uF
- C2: value 50uF -> 47uF
Changed lines of the file:
@@
 LIBS:contrib
 LIBS:valves
+LIBS:Single_transistor_AMP_miculis-cache
 EELAYER 25 0
 EELAYER END
@@
 F 1 "4.7k" V 4400 2200 50  0000 C CNN
 F 2 "Resistors_THT:R_Axial_DIN0204_L3.6mm_D1.6mm_P7.62mm_Horizontal" V 4330 2200 50  0001 C CNN
-F 3 "" H 4400 2200 50  0001 C CNN
+F 3 "http://www.farnell.com/datasheets/168591.pdf?_ga=2.16783033.127273279.1528788908-352338308.1521105712&_gac=1.15016706.1528660445.EAIaIQobChMIs6eo8-_J2wIVHJSyCh0a5gCjEAAYASAAEgLzUPD_BwE" H 4400 2200 50  0001 C CNN
 	1    4400 2200
 	1    0    0    -1
@@
 F 1 "1.8k" V 4400 3200 50  0000 C CNN
 F 2 "Resistors_THT:R_Axial_DIN0204_L3.6mm_D1.6mm_P7.62mm_Horizontal" V 4330 3200 50  0001 C CNN
-F 3 "" H 4400 3200 50  0001 C CNN
+F 3 "http://www.farnell.com/datasheets/2045734.pdf?_ga=2.11342260.127273279.1528788908-352338308.1521105712&_gac=1.37039764.1528660445.EAIaIQobChMIs6eo8-_J2wIVHJSyCh0a5gCjEAAYASAAEgLzUPD_BwE" H 4400 3200 50  0001 C CNN
 	1    4400 3200
 	1    0    0    -1
@@
 F 1 "6.8k" V 3800 3200 50  0000 C CNN
 F 2 "Resistors_THT:R_Axial_DIN0204_L3.6mm_D1.6mm_P7.62mm_Horizontal" V 3730 3200 50  0001 C CNN
-F 3 "" H 3800 3200 50  0001 C CNN
+F 3 "http://www.farnell.com/datasheets/1716725.pdf?_ga=2.37606944.127273279.1528788908-352338308.1521105712&_gac=1.2822020.1528660445.EAIaIQobChMIs6eo8-_J2wIVHJSyCh0a5gCjEAAYASAAEgLzUPD_BwE" H 3800 3200 50  0001 C CNN
 	1    3800 3200
 	1    0    0    -1
@@
 F 1 "22k" V 3800 2200 50  0000 C CNN
 F 2 "Resistors_THT:R_Axial_DIN0204_L3.6mm_D1.6mm_P7.62mm_Horizontal" V 3730 2200 50  0001 C CNN
-F 3 "" H 3800 2200 50  0001 C CNN
+F 3 "http://www.farnell.com/datasheets/1723855.pdf?_ga=2.72225043.127273279.1528788908-352338308.1521105712&_gac=1.6606342.1528660445.EAIaIQobChMIs6eo8-_J2wIVHJSyCh0a5gCjEAAYASAAEgLzUPD_BwE" H 3800 2200 50  0001 C CNN
 	1    3800 2200
 	1    0    0    -1
@@
 F 1 "BC548" H 4500 2650 50  0000 L CNN
 F 2 "TO_SOT_Packages_THT:TO-92_Inline_Narrow_Oval" H 4500 2575 50  0001 L CIN
-F 3 "ateeja.lv/tranis" H 4300 2650 50  0001 L CNN
+F 3 "http://www.farnell.com/datasheets/2299482.pdf?_ga=2.252182025.127273279.1528788908-352338308.1521105712&_gac=1.49614610.1528660445.EAIaIQobChMIs6eo8-_J2wIVHJSyCh0a5gCjEAAYASAAEgLzUPD_BwE" H 4300 2650 50  0001 L CNN
 	1    4300 2650
 	1    0    0    -1
@@
 F 1 "Conn_01x02" H 2900 2550 50  0000 C CNN
 F 2 "Pin_Headers:Pin_Header_Straight_1x02_Pitch2.54mm" H 2900 2750 50  0001 C CNN
-F 3 "" H 2900 2750 50  0001 C CNN
+F 3 "http://www.farnell.com/da" H 2900 2750 50  0001 C CNN
 	1    2900 2750
 	-1   0    0    1
@@
 F 1 "Conn_01x02" H 5750 2200 50  0000 C CNN
 F 2 "Connectors_Terminal_Blocks:TerminalBlock_bornier-2_P5.08mm" H 5750 2400 50  0001 C CNN
-F 3 "" H 5750 2400 50  0001 C CNN
+F 3 "http://www.farnell.com/da" H 5750 2400 50  0001 C CNN
 	1    5750 2400
 	1    0    0    -1
@@
 P 3450 2650
 F 0 "C1" H 3460 2720 50  0000 L CNN
-F 1 "20uF" H 3460 2570 50  0000 L CNN
+F 1 "22uF" H 3460 2570 50  0000 L CNN
 F 2 "Capacitors_THT:CP_Radial_D6.3mm_P2.50mm" H 3450 2650 50  0001 C CNN
-F 3 "" H 3450 2650 50  0001 C CNN
+F 3 "http://www.farnell.com/datasheets/2321915.pdf?_ga=2.243727749.127273279.1528788908-352338308.1521105712&_gac=1.177400337.1528660445.EAIaIQobChMIs6eo8-_J2wIVHJSyCh0a5gCjEAAYASAAEgLzUPD_BwE" H 3450 2650 50  0001 C CNN
 	1    3450 2650
 	0    -1   -1   0
@@
 P 4700 3200
 F 0 "C2" H 4710 3270 50  0000 L CNN
-F 1 "50uF" H 4710 3120 50  0000 L CNN
+F 1 "47uF" H 4710 3120 50  0000 L CNN
 F 2 "Capacitors_THT:CP_Radial_D7.5mm_P2.50mm" H 4700 3200 50  0001 C CNN
-F 3 "" H 4700 3200 50  0001 C CNN
+F 3 "http://www.farnell.com/datasheets/2322165.pdf?_ga=2.71178896.127273279.1528788908-352338308.1521105712&_gac=1.149154306.1528660445.EAIaIQobChMIs6eo8-_J2wIVHJSyCh0a5gCjEAAYASAAEgLzUPD_BwE" H 4700 3200 50  0001 C CNN
 	1    4700 3200
 	1    0    0    -1
@@
 P 5100 2400
 F 0 "C3" H 5110 2470 50  0000 L CNN
-F 1 "20uF" H 5110 2320 50  0000 L CNN
+F 1 "22uF" H 5110 2320 50  0000 L CNN
 F 2 "Capacitors_THT:CP_Radial_D6.3mm_P2.50mm" H 5100 2400 50  0001 C CNN
-F 3 "" H 5100 2400 50  0001 C CNN
+F 3 "http://www.farnell.com/datasheets/2321915.pdf?_ga=2.243727749.127273279.1528788908-352338308.1521105712&_gac=1.177400337.1528660445.EAIaIQobChMIs6eo8-_J2wIVHJSyCh0a5gCjEAAYASAAEgLzUPD_BwE" H 5100 2400 50  0001 C CNN
 	1    5100 2400
 	0    -1   -1   0
